File: CH340E.kicad_sch (KiCad schematic)
At the start: 3 parts, among them U4 CH340E

Commit message: feat(hardware): add KLC compliance properties and supplier metadata to schematic components
Adds KiCad Library Convention properties (KLC_S3.3, KLC_S4.1) to multiple components for compliance, and includes manufacturer, part number, and distributor links (Mouser, DigiKey, LCSC) to the CH340E USB-to-serial converter component.
Parts:
- U4: Distributor Link 1 (none) -> https://eu.mouser.com/ProductDetail/Adafruit/5893?qs=jRuttq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; Distributor Link 2 (none) -> https://www.digikey.com/en/products/detail/sparkfun-electro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; LCSC (none) -> C99652; Manufacturer (none) -> Adafruit; Manufacturer part Number (none) -> 5893
Changed lines of the file:
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@@
+			)
+		)
+		(property "KLC_S3.3" ""
+			(at 54.61 59.69 0)
+			(effects
+				(font
+					(size 1.27 1.27)
+				)
+				(hide yes)
+			)
+		)
+		(property "KLC_S4.1" ""
+			(at 54.61 59.69 0)
+			(effects
+				(font
+					(size 1.27 1.27)
+				)
+				(hide yes)
 			)
 		)
@@
 			)
 		)
+		(property "KLC_S3.3" ""
+			(at 44.45 59.69 0)
+			(effects
+				(font
+					(size 1.27 1.27)
+				)
+				(hide yes)
+			)
+		)
+		(property "KLC_S4.1" ""
+			(at 44.45 59.69 0)
+			(effects
+				(font
+					(size 1.27 1.27)
+				)
+				(hide yes)
+			)
+		)
 		(pin "1"
 		)
@@
 			(at 78.74 72.39 0)
 			(effects
+				(font
+					(size 1.27 1.27)
+				)
+				(hide yes)
+			)
+		)
+		(property "Manufacturer" "Adafruit"
+			(at 78.74 72.39 0)
+			(effects
+				(font
+					(size 1.27 1.27)
+				)
+				(hide yes)
+			)
+		)
+		(property "Manufacturer part Number" "5893"
+			(at 78.74 72.39 0)
+			(effects
+				(font
+					(size 1.27 1.27)
+				)
+				(hide yes)
+			)
+		)
+		(property "Distributor Link 1" "https://eu.mouser.com/ProductDetail/Adafruit/5893?qs=jRuttqqUwMS7meI7BJ44ng%3D%3D"
+			(at 78.74 72.39 0)
+			(effects
+				(font
+					(size 1.27 1.27)
+				)
+				(hide yes)
+			)
+		)
+		(property "Distributor Link 2" "https://www.digikey.com/en/products/detail/sparkfun-electronics/16278/17829769?s=N4IgTCBcDaIMIAkDMAWADAURAXQL5A"
+			(at 78.74 72.39 0)
+			(effects
+				(font
+					(size 1.27 1.27)
+				)
+				(hide yes)
+			)
+		)
+		(property "LCSC" "C99652"
+			(at 78.74 72.39 0)
+			(effects
+				(font
+					(size 1.27 1.27)
+				)
+				(hide yes)
+			)
+		)
+		(property "KLC_S3.3" ""
+			(at 78.74 72.39 0)
+			(effects
+				(font
+					(size 1.27 1.27)
+				)
+				(hide yes)
+			)
+		)
+		(property "KLC_S4.1" ""
+			(at 78.74 72.39 0)
+			(effects
